File: ur10.kicad_pcb (KiCad board)
At the start: 2 copper layers, 65 x 35 mm, 18 parts, among them K1 TNA-2C-12-05-L, Q1 AO3401A

Commit message: Use THT jumpers instead of solder jumpers.
Reason: they are visible from top side.
Parts:
- JP1, JP2, JP3: footprint Jumper:SolderJumper-2_P1.3mm_Open_RoundedPad1.0x1.5mm -> Connector_PinHeader_2.54mm:PinHeader_1x02_P2.54mm_Vertical; moved to F.Cu
- moved JP2 20.1 mm to (156.0, 103.1), turned to 0 degrees
- moved JP1 14.7 mm to (160.0, 105.7)
- moved D3 2.59 mm to (114.6, 105.9)
- moved JP3 1.53 mm to (109.5, 113.0), turned to 180 degrees
Routing:
- net /12: track 18.4 -> 37.0 mm
- net /22: track 36.2 -> 53.6 mm
- net /14: track 37.3 -> 27.7 mm
- net /24: track 29.6 -> 37.3 mm
- net Net-(D3-K): track 4.96 -> 6.40 mm
- net Net-(D2-K): track 21.1 -> 20.2 mm
- net /21: track 27.9 -> 28.8 mm
